File: electrical/base board/file61980A01.sch (KiCad schematic (older format))
At the start: 17 parts, among them J701 PTC thermistor, J702 PTC thermistor, J703 PTC thermistor, J704 PTC thermistor, J705 water sensor, J706 IMU

Commit message: updated sub board
Parts:
- removed J705: water sensor, symbol Connector_Generic:Conn_01x02
- removed J706: IMU, symbol Connector_Generic:Conn_01x04
- removed R705: 1.0M, symbol Device:R_Small_US
- removed R706, R707: 100K, symbol Device:R_Small_US
- renumbered C701 to C?, C702 to C?, C703 to C?, C704 to C?, J701 to J?, J702 to J?, J703 to J?, J704 to J?, R701 to R?, R702 to R?, R703 to R?, R704 to R?
Connections:
- net labels removed: scl, sda, water
- wire segments 27 -> 20
