File: electrical/sub board/board/ESC_servo_lights.sch (KiCad schematic (older format))
At the start: 27 parts

Commit message: updated sub board
Parts:
- removed D?: BZX84C11, symbol Device:D_Zener
- added C901, C902, C905: 4.7uF, Capacitor_SMD:C_0603_1608Metric, symbol Device:C_Small
- added C903, C904, C906: 0.1uF, Capacitor_SMD:C_0402_1005Metric, symbol Device:C_Small
- added C908: 0.1uF,25V, Capacitor_SMD:C_01005_0402Metric, symbol Device:C_Small
- C907: renamed from C?; value 10uF, 25V -> 10uF,25V; footprint (none) -> Capacitor_SMD:C_1206_3216Metric
- C909: renamed from C?; value 0.01uF, 16V -> 10nF, 16V; footprint (none) -> Capacitor_SMD:C_0402_1005Metric
- C910, C911: renamed from C?; value 1uF, 16V -> 1.0uF, 16V; footprint (none) -> Capacitor_SMD:C_0603_1608Metric
- D901: renamed from D?; value CMDSH-3 -> RB720M-30; footprint (none) -> Diode_SMD:SOD-923
- D902: renamed from D?; value SS13 -> 30V, 1A; footprint (none) -> Diode_SMD:DO-219AD
- J901: renamed from J?; value Conn_01x03 -> thruster_esc0; footprint (none) -> Connector_PinHeader_2.54mm:PinHeader_1x03_P2.54mm_Vertical
- J902: renamed from J?; value Conn_01x03 -> thruster_esc1; footprint (none) -> Connector_PinHeader_2.54mm:PinHeader_1x03_P2.54mm_Vertical
- J903: renamed from J?; value Conn_01x03 -> thruster_esc2; footprint (none) -> Connector_PinHeader_2.54mm:PinHeader_1x03_P2.54mm_Vertical
- J904: renamed from J?; value Conn_01x03 -> thruster_esc3; footprint (none) -> Connector_PinHeader_2.54mm:PinHeader_1x03_P2.54mm_Vertical
- J905: renamed from J?; value Conn_01x03 -> thruster_esc4; footprint (none) -> Connector_PinHeader_2.54mm:PinHeader_1x03_P2.54mm_Vertical
- J906: renamed from J?; value Conn_01x03 -> thruster_esc5; footprint (none) -> Connector_PinHeader_2.54mm:PinHeader_1x03_P2.54mm_Vertical
- J907: renamed from J?; value Conn_01x03 -> thruster_esc6; footprint (none) -> Connector_PinHeader_2.54mm:PinHeader_1x03_P2.54mm_Vertical
- J908: renamed from J?; value Conn_01x03 -> thruster_esc7; footprint (none) -> Connector_PinHeader_2.54mm:PinHeader_1x03_P2.54mm_Vertical
- J909: renamed from J?; value Conn_01x03 -> servo0; footprint (none) -> Connector_PinHeader_2.54mm:PinHeader_1x03_P2.54mm_Vertical
- J910: renamed from J?; value Conn_01x03 -> servo1; footprint (none) -> Connector_PinHeader_2.54mm:PinHeader_1x03_P2.54mm_Vertical
- J911: renamed from J?; value Conn_01x03 -> servo2; footprint (none) -> Connector_PinHeader_2.54mm:PinHeader_1x03_P2.54mm_Vertical
- J912: renamed from J?; value Conn_01x03 -> servo3; footprint (none) -> Connector_PinHeader_2.54mm:PinHeader_1x03_P2.54mm_Vertical
- J913: renamed from J?; value Conn_01x02 -> LED; footprint (none) -> Connector_Hirose:Hirose_DF13C_CL535-0402-2-51_1x02-1MP_P1.25mm_Vertical
- L901: renamed from L?; footprint (none) -> Inductor_SMD:L_TDK_VLS3012
- R901: renamed from R?; footprint (none) -> Resistor_SMD:R_0402_1005Metric
- R902: renamed from R?; footprint (none) -> Resistor_SMD:R_0805_2012Metric
- U901, U902, U903: renamed from U?; footprint (none) -> Package_SO:SO-14_3.9x8.65mm_P1.27mm
- U904: renamed from U?; footprint (none) -> sub:VSSOP-8_3.0x3.0mm_P0.65mm-EP
Connections:
- net +5V: now also D901.2 (A), C901.1, C902.1, C903.1, C904.1, C905.1, C906.1
- net +BATT: now also C908.1
- net GND: now also C901.2, C902.2, C903.2, C904.2, C905.2, C906.2, C908.2
Other:
- note removed: "Check Zener diode V\n"
- moved on the sheet: C907, D901
