File: electrical/sub board/board/RS485.sch (KiCad schematic (older format))
At the start: 7 parts

Commit message: updated sub board
Parts:
- C301, C302: renamed from C?; footprint (none) -> Capacitor_SMD:C_0402_1005Metric
- C303: renamed from C?; footprint (none) -> Capacitor_SMD:C_0603_1608Metric
- J301: renamed from J?; footprint (none) -> Connector_Hirose:Hirose_DF13C_CL535-0402-2-51_1x02-1MP_P1.25mm_Vertical
- R301: renamed from R?; footprint (none) -> Resistor_SMD:R_0402_1005Metric
- R302: renamed from R?; footprint (none) -> Resistor_SMD:R_1206_3216Metric
- U301: renamed from U?; footprint (none) -> Package_DFN_QFN:DFN-10-1EP_3x3mm_P0.5mm_EP1.55x2.48mm
Changed lines of the file:
@@
 $Descr A4 11693 8268
 encoding utf-8
-Sheet 3 12
+Sheet 3 14
 Title ""
 Date ""
@@
 $EndDescr
 $Comp
-L sub_board:MAX22500E U?
+L sub_board:MAX22500E U301
 U 1 1 61678045
 P 5750 3500
-F 0 "U?" H 6100 4300 50  0000 L CNN
+F 0 "U301" H 6100 4300 50  0000 L CNN
 F 1 "MAX22500E" H 6100 4200 50  0000 L CNN
-F 2 "" H 5750 3500 50  0001 C CNN
-F 3 "" H 5750 3500 50  0001 C CNN
+F 2 "Package_DFN_QFN:DFN-10-1EP_3x3mm_P0.5mm_EP1.55x2.48mm" H 5750 3500 50  0001 C CNN
+F 3 "MAX22500EATB+-ND" H 5750 3500 50  0001 C CNN
 	1    5750 3500
 	1    0    0    -1
 $EndComp
 $Comp
-L power:+3.3V #PWR?
+L power:+3.3V #PWR0304
 U 1 1 61678ABE
 P 5700 2750
-F 0 "#PWR?" H 5700 2600 50  0001 C CNN
+F 0 "#PWR0304" H 5700 2600 50  0001 C CNN
 F 1 "+3.3V" H 5715 2923 50  0000 C CNN
 F 2 "" H 5700 2750 50  0001 C CNN
@@
 $EndComp
 $Comp
-L power:GND #PWR?
+L power:GND #PWR0305
 U 1 1 61678FF3
 P 5700 4050
-F 0 "#PWR?" H 5700 3800 50  0001 C CNN
+F 0 "#PWR0305" H 5700 3800 50  0001 C CNN
 F 1 "GND" H 5705 3877 50  0000 C CNN
 F 2 "" H 5700 4050 50  0001 C CNN
@@
 Connection ~ 5700 2750
 $Comp
-L Device:R_Small_US R?
+L Device:R_Small_US R302
 U 1 1 6167952F
 P 6600 3350
-F 0 "R?" H 6668 3396 50  0000 L CNN
+F 0 "R302" H 6668 3396 50  0000 L CNN
 F 1 "120R" H 6668 3305 50  0000 L CNN
-F 2 "" H 6600 3350 50  0001 C CNN
-F 3 "~" H 6600 3350 50  0001 C CNN
+F 2 "Resistor_SMD:R_1206_3216Metric" H 6600 3350 50  0001 C CNN
+F 3 "A129799CT-ND" H 6600 3350 50  0001 C CNN
 	1    6600 3350
 	1    0    0    -1
@@
 	6600 3250 7400 3250
 $Comp
-L Device:R_Small_US R?
+L Device:R_Small_US R301
 U 1 1 6167AC91
 P 5150 4050
-F 0 "R?" H 5218 4096 50  0000 L CNN
+F 0 "R301" H 5218 4096 50  0000 L CNN
 F 1 "40K" H 5218 4005 50  0000 L CNN
-F 2 "" H 5150 4050 50  0001 C CNN
-F 3 "~" H 5150 4050 50  0001 C CNN
+F 2 "Resistor_SMD:R_0402_1005Metric" H 5150 4050 50  0001 C CNN
+F 3 "RMCF0402FT40R2CT-ND" H 5150 4050 50  0001 C CNN
 	1    5150 4050
 	1    0    0    -1
@@
 	5150 3950 5150 3800
 $Comp
-L power:GND #PWR?
+L power:GND #PWR0301
 U 1 1 6167B4EA
 P 5150 4150
-F 0 "#PWR?" H 5150 3900 50  0001 C CNN
+F 0 "#PWR0301" H 5150 3900 50  0001 C CNN
 F 1 "GND" H 5155 3977 50  0000 C CNN
 F 2 "" H 5150 4150 50  0001 C CNN
@@
 $EndComp
 $Comp
-L Device:C_Small C?
+L Device:C_Small C301
 U 1 1 6167B911
 P 5300 1900
-F 0 "C?" H 5392 1946 50  0000 L CNN
+F 0 "C301" H 5392 1946 50  0000 L CNN
 F 1 "0.1uF" H 5392 1855 50  0000 L CNN
-F 2 "" H 5300 1900 50  0001 C CNN
-F 3 "~" H 5300 1900 50  0001 C CNN
+F 2 "Capacitor_SMD:C_0402_1005Metric" H 5300 1900 50  0001 C CNN
+F 3 "478-11506-1-ND" H 5300 1900 50  0001 C CNN
 	1    5300 1900
 	1    0    0    -1
 $EndComp
 $Comp
-L Device:C_Small C?
+L Device:C_Small C302
 U 1 1 6167BE53
 P 5700 1900
-F 0 "C?" H 5792 1946 50  0000 L CNN
+F 0 "C302" H 5792 1946 50  0000 L CNN
 F 1 "0.1uF" H 5792 1855 50  0000 L CNN
-F 2 "" H 5700 1900 50  0001 C CNN
-F 3 "~" H 5700 1900 50  0001 C CNN
+F 2 "Capacitor_SMD:C_0402_1005Metric" H 5700 1900 50  0001 C CNN
+F 3 "478-11506-1-ND" H 5700 1900 50  0001 C CNN
 	1    5700 1900
 	1    0    0    -1
@@
 	5700 1800 5300 1800
 $Comp
-L power:+3.3V #PWR?
+L power:+3.3V #PWR0302
 U 1 1 6167C3BB
 P 5300 1800
-F 0 "#PWR?" H 5300 1650 50  0001 C CNN
+F 0 "#PWR0302" H 5300 1650 50  0001 C CNN
 F 1 "+3.3V" H 5315 1973 50  0000 C CNN
 F 2 "" H 5300 1800 50  0001 C CNN
@@
 Connection ~ 5300 1800
 $Comp
-L power:GND #PWR?
+L power:GND #PWR0303
 U 1 1 6167C7EA
 P 5300 2000
-F 0 "#PWR?" H 5300 1750 50  0001 C CNN
+F 0 "#PWR0303" H 5300 1750 50  0001 C CNN
 F 1 "GND" H 5305 1827 50  0000 C CNN
 F 2 "" H 5300 2000 50  0001 C CNN
@@
 Connection ~ 5300 2000
 $Comp
-L Device:C_Small C?
+L Device:C_Small C303
 U 1 1 6167CD48
 P 6100 1900
-F 0 "C?" H 6192 1946 50  0000 L CNN
+F 0 "C303" H 6192 1946 50  0000 L CNN
 F 1 "4.7uF" H 6192 1855 50  0000 L CNN
-F 2 "" H 6100 1900 50  0001 C CNN
-F 3 "~" H 6100 1900 50  0001 C CNN
+F 2 "Capacitor_SMD:C_0603_1608Metric" H 6100 1900 50  0001 C CNN
+F 3 "1276-1044-1-ND" H 6100 1900 50  0001 C CNN
 	1    6100 1900
 	1    0    0    -1
@@
 	5150 3500 4600 3500
 $Comp
-L Connector_Generic:Conn_01x02 J?
+L Connector_Generic:Conn_01x02 J301
 U 1 1 6167E7CB
 P 7600 3300
-F 0 "J?" H 7680 3292 50  0000 L CNN
+F 0 "J301" H 7680 3292 50  0000 L CNN
 F 1 "RS485" H 7680 3201 50  0000 L CNN
-F 2 "" H 7600 3300 50  0001 C CNN
-F 3 "~" H 7600 3300 50  0001 C CNN
+F 2 "Connector_Hirose:Hirose_DF13C_CL535-0402-2-51_1x02-1MP_P1.25mm_Vertical" H 7600 3300 50  0001 C CNN
+F 3 "H126391-ND" H 7600 3300 50  0001 C CNN
 	1    7600 3300
 	1    0    0    -1
