File: electrical/sub board/board/RaspberryPiCM3+.sch (KiCad schematic (older format))
At the start: 11 parts

Commit message: updated sub board
Parts:
- removed U?: RaspberryPi-CM3+, symbol MCU_Module:RaspberryPi-CM3+
- added C801: 4.7uF, Capacitor_SMD:C_0603_1608Metric, symbol Device:C_Small
- added U801: RaspberryPi-CM3+L, Connector:Conn_TE-DDR2-SODIMM-0.6-200P-doublesided, symbol MCU_Module:RaspberryPi-CM3+L
- J801: renamed from J?; footprint (none) -> Connector_USB:USB_Micro-B_Wuerth_629105150521
- J802, J804: renamed from J?; footprint (none) -> sub:Molex_200528-0150_1x15-1MP_P1.00mm_Horizontal
- J803: renamed from J?; footprint (none) -> sub:MEM2061
- R801, R802, R803, R804, R805, R806: renamed from R?; footprint (none) -> Resistor_SMD:R_0402_1005Metric
Connections:
- net labels removed: sd_cd, spi_miso, spi_mosi, spi_ncs, spi_sclk
- wire segments 84 -> 76
- no-connect marks 1 -> 2
Other:
- note added: "Check camera connector and orientation"
- note added: "route USB as 90ohm diff\n"
- note added: "run as 100ohm diff\n"
