File: electrical/sub board/board/battery.sch (KiCad schematic (older format))
At the start: 8 parts

Commit message: updated sub board
Parts:
- added R401: 4.7K, Resistor_SMD:R_0402_1005Metric, symbol Device:R_Small_US
- BT401: renamed from BT?; footprint (none) -> sub:AMASS_XT60-M
- C401: renamed from C?; value C_Small -> 1.0uF, 16V; footprint (none) -> Capacitor_SMD:C_0603_1608Metric
- J401, J402, J403, J404: renamed from J?; value Conn_01x02 -> thruster_esc; footprint (none) -> sub:AMASS_XT30U-F_1x02_P5.0mm_Vertical
- R402: renamed from R?; footprint (none) -> Resistor_SMD:R_Shunt_Yaego_PU3921
- U401: renamed from U?; footprint (none) -> Package_DFN_QFN:DFN-8-1EP_3x3mm_P0.5mm_EP1.66x2.38mm
Connections:
- net alcc: now also R401.1
- new net +3V3: R401.2
Other:
- note added: "https://hobbyking.com/en_us/turnigy-2200mah-2s-25c-lipo-pack-w-xt60.html?queryID=53fd6d95b7331c8d18e1cd91f698c5dd&objectID=74814&indexName=hbk_live_products_analytics"
