File: electrical/sub board/board/board.sch (KiCad schematic (older format))
At the start: 6 parts

Commit message: updated sub board
Parts:
- F101: renamed from F?; value Polyfuse_Small -> 6A; footprint (none) -> sub:2920L
- R101, R102, R103, R104: renamed from R?; footprint (none) -> Resistor_SMD:R_0402_1005Metric
- R105: renamed from R?; footprint (none) -> sub:AMASS_XT30U-F_1x02_P5.0mm_Vertical
Other:
- note added: "Power switch\n"
- moved on the sheet: R101, R102, R103, R104
