File: electrical/sub board/board/ethernet.sch (KiCad schematic (older format))
At the start: 26 parts

Commit message: updated sub board
Parts:
- added C208, C209: 10uF, Capacitor_SMD:C_0805_2012Metric, symbol Device:C_Small
- added R201, R202, R203, R204: 2.2K, Resistor_SMD:R_0402_1005Metric, symbol Device:R_Small_US
- C201: renamed from C?; value 0.01uF -> 10nF, 16V; footprint (none) -> Capacitor_SMD:C_0402_1005Metric
- C202, C203: renamed from C?; value 10nF -> 10nF, 16V; footprint (none) -> Capacitor_SMD:C_0402_1005Metric
- C204, C205: renamed from C?; footprint (none) -> Capacitor_SMD:C_0402_1005Metric
- C206, C207, C212, C213: renamed from C?; footprint (none) -> Capacitor_SMD:C_0603_1608Metric
- C210, C211: renamed from C?; value 230nF -> 220nF,16V; footprint (none) -> Capacitor_SMD:C_0603_1608Metric
- D201, D202, D203: renamed from D?; footprint (none) -> LED_SMD:LED_0402_1005Metric
- FB201, FB202: renamed from FB?; footprint (none) -> Resistor_SMD:R_0603_1608Metric
- FL201: renamed from FL?; footprint (none) -> Inductor_SMD:L_WE_SL5
- J201: renamed from J?; footprint (none) -> Connector_Hirose:Hirose_DF13C_CL535-0402-2-51_1x02-1MP_P1.25mm_Vertical
- R205, R208, R209, R210, R211: renamed from R?; footprint (none) -> Resistor_SMD:R_0402_1005Metric
- R206, R207: renamed from R?; footprint (none) -> Resistor_SMD:R_2512_6332Metric
- U201: renamed from U?; footprint (none) -> Package_DFN_QFN:TQFN-32-1EP_5x5mm_P0.5mm_EP2.1x2.1mm
Connections:
- net +3V3: now also R201.2, R202.2, R204.2
- net GND: now also C208.2, C209.2, R203.1
- net crs_dv: now also R201.1
- net mdio: now also R204.1
- net rx_d0: now also R203.2
- net rx_d1: now also R202.1
- net at C203.1, C205.1, C207.1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: now also C209.1
- net at C202.1, C204.1, C206.1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: now also C208.1
- no-connect marks 3 -> 6
Other:
- note added: "100ohm differential"
- note added: "50ohm SE\n"
- note added: "Straps\n"
- moved on the sheet: C202, C203, C204, C205, C206, C207
