File: electrical/sub board/board/internal_sensors.sch (KiCad schematic (older format))
At the start: 18 parts

Commit message: updated sub board
Parts:
- removed R? (x2): 100K, symbol Device:R_Small_US
- removed U?: TLV7011, symbol sub_board:TLV7011
- added C705: 4.7uF, Capacitor_SMD:C_0603_1608Metric, symbol Device:C_Small
- added C706: 0.1uF, Capacitor_SMD:C_0402_1005Metric, symbol Device:C_Small
- added J706: water sensor1, Connector_Hirose:Hirose_DF13C_CL535-0402-2-51_1x02-1MP_P1.25mm_Vertical, symbol Connector_Generic:Conn_01x02
- added R706, R708, R709, R710: 1.0K, Resistor_SMD:R_0402_1005Metric, symbol Device:R_Small_US
- added R707: 1.0M, Resistor_SMD:R_0402_1005Metric, symbol Device:R_Small_US
- added U701: TLV4082, Package_TO_SOT_SMD:SOT-23-6, symbol sub_board:TLV4082
- C701, C702, C703, C704: renamed from C?; value 1.0uF -> 1.0uF, 16V; footprint (none) -> Capacitor_SMD:C_0603_1608Metric
- J701, J702, J703, J704: renamed from J?; footprint (none) -> Connector_Hirose:Hirose_DF13C_CL535-0402-2-51_1x02-1MP_P1.25mm_Vertical
- J705: renamed from J?; value water sensor -> water sensor0; footprint (none) -> Connector_Hirose:Hirose_DF13C_CL535-0402-2-51_1x02-1MP_P1.25mm_Vertical
- J707: renamed from J?; footprint (none) -> Connector_Hirose:Hirose_DF13C_CL535-0404-8-51_1x04-1MP_P1.25mm_Vertical
- R701, R702, R703, R704: renamed from R?; value SOT -> 10K; footprint (none) -> Resistor_SMD:R_0402_1005Metric
- R705: renamed from R?; footprint (none) -> Resistor_SMD:R_0402_1005Metric
Connections:
- net +3V3: now also C705.1, C706.1, R707.2, U701.1 (Vcc)
- net GND: now also C705.2, C706.2, R706.1, R708.1, U701.5 (gnd); no longer J705.2 (Pin_2)
- net water: now also U701.2 (out1), U701.3 (out2)
- net at J705.1 (Pin_1), R705.1: now also R709.1
- new net: J705.2 (Pin_2), R706.2
- new net: R710.1, U701.4 (in2)
- new net: R709.2, U701.6 (in1)
- new net: J706.1 (Pin_1), R707.1, R710.2
- new net: J706.2 (Pin_2), R708.2
