File: electrical/sub board/board/micro.sch (KiCad schematic (older format))
At the start: 36 parts

Commit message: updated sub board
Parts:
- removed J? (x2): USB_B_Micro, symbol Connector:USB_B_Micro
- removed X?: ASE-13MHz, Oscillator:Oscillator_SMD_Abracon_ASE-4Pin_3.2x2.5mm, symbol Oscillator:ASE-xxxMHz
- added C1326: 2.2uF, Capacitor_SMD:C_0603_1608Metric, symbol Device:C_Small
- added C1327, C1328, C1329: 0.1uF, Capacitor_SMD:C_0402_1005Metric, symbol Device:C_Small
- added C1330: 4.7uF, Capacitor_SMD:C_0603_1608Metric, symbol Device:C_Small
- added J1301, J1302: USB_B_Micro, Connector_USB:USB_Micro-B_Wuerth_629105150521, symbol Connector:USB_B_Micro
- added R1303: 10K, Resistor_SMD:R_0402_1005Metric, symbol Device:R_Small_US
- added X1301: 13MHz, sub:831056290, symbol Oscillator:ASE-xxxMHz
- C1301, C1303, C1305, C1307, C1309, C1310, C1311, C1312, C1313, C1314, C1315, C1317, C1318, C1319, C1320, C1324, C1325: renamed from C?; footprint (none) -> Capacitor_SMD:C_0402_1005Metric
- C1302, C1304, C1306, C1308, C1316, C1321, C1322: renamed from C?; footprint (none) -> Capacitor_SMD:C_0603_1608Metric
- C1323: renamed from C?; value 1.0uF -> 1.0uF, 16V; footprint (none) -> Capacitor_SMD:C_0603_1608Metric
- D1301: renamed from D?; footprint (none) -> LED_SMD:LED_0402_1005Metric
- J1303: renamed from J?; footprint (none) -> Connector_IDC:IDC-Header_2x10_P2.54mm_Vertical
- J1304: renamed from J?; footprint (none) -> sub:MEM2061
- R1301: renamed from R?; footprint (none) -> Resistor_SMD:R_0402_1005Metric
- R1302: renamed from R?; value 330R -> 470R; footprint (none) -> Resistor_SMD:R_0402_1005Metric
- U1301: renamed from U?; footprint (none) -> sub:QFN-24-1EP_4x4mm_P0.5mm_EP2.6x2.6mm
- X1302: renamed from X?; value ASE-25MHz -> 25MHz; footprint Oscillator:Oscillator_SMD_Abracon_ASE-4Pin_3.2x2.5mm -> sub:ASFL1
- gave numbers to parts that had none: 1
Connections:
- net GND is gone; now on net +3V3: C1301.2, C1302.2, C1303.2, C1304.2, C1305.2, C1306.2, C1307.2, C1308.2, C1309.2, C1310.2, C1311.2, C1312.2, C1313.2, C1314.2, C1315.2, C1316.2, C1317.2, C1318.2, C1319.2, C1320.2, C1321.2, C1322.2, C1323.2, C1324.2, C1325.2, J1303.10 (Pin_10), J1303.12 (Pin_12), J1303.14 (Pin_14), J1303.16 (Pin_16), J1303.18 (Pin_18), J1303.20 (Pin_20), J1303.4 (Pin_4), J1303.6 (Pin_6), J1303.8 (Pin_8), J1304.11 (SHIELD), J1304.6 (VSS), R1301.1, U1301.25 (gnd), U1302.102 (VSS), U1302.113 (VSS), U1302.126 (VSS), U1302.135 (VSS), U1302.14 (VSS), U1302.148 (VSS), U1302.158 (VSS), U1302.166 (BOOT0), U1302.22 (VSS), U1302.37 (VSSA), U1302.48 (VSS), U1302.61 (VSS), U1302.71 (VSS), U1302.90 (VSS), X1302.2 (GND)
- net +1V8: now also C1328.2
- net +3V3: now also C1326.1, C1327.1, C1327.2, C1328.1, C1329.1, C1329.2, C1330.1, C1330.2, J1301.5 (GND), J1301.6 (Shield), J1302.5 (GND), J1302.6 (Shield), X1301.2 (GND), X1301.4 (Vdd)
- net fs_dm: now also J1302.2 (D-)
- net fs_dp: now also J1302.3 (D+)
- net fs_vbus: now also J1302.1 (VBUS)
- net lidar_rx: now reaches U1302.121 (PA10)
- net at U1301.5 (dm): now also J1301.2 (D-)
- net at U1301.6 (dp): now also J1301.3 (D+)
- net at U1301.23 (refclk): now also X1301.3 (OUT)
- net +5V: no longer names the net of U1301.2 (VBus)
- net +5V: now also R1303.1
- net scl0 renamed lidar_tx
- net sda0 renamed lidar_pwr
- new net: C1326.2, J1301.1 (VBUS), R1303.2
Other:
- moved on the sheet: C1323, C1324
