File: electrical/sub board/board/water_sensors.sch (KiCad schematic (older format))
At the start: 39 parts

Commit message: updated sub board
Parts:
- removed C?: 22uF, 25V, symbol Device:C_Small
- removed J?: depth, symbol Connector_Generic:Conn_01x02
- removed J?: pinger, symbol Connector_Generic:Conn_01x02
- removed R? (x2): 4.7K, symbol Device:R_Small_US
- added C1201, C1218: 10uF,25V, Capacitor_SMD:C_1206_3216Metric, symbol Device:C_Small
- added C1207, C1209: 1nF, Capacitor_SMD:C_0402_1005Metric, symbol Device:C_Small
- added C1213: 6.8nF, Capacitor_SMD:C_0402_1005Metric, symbol Device:C_Small
- added C1217: SOT, Capacitor_SMD:C_0402_1005Metric, symbol Device:C_Small
- added C1219: 10uF, 63V, X7R, Capacitor_SMD:C_1210_3225Metric, symbol Device:C_Small
- added F1201, F1202: 3A, sub:2016, symbol Device:Polyfuse_Small
- added J1203: Transducers, Connector_Hirose:Hirose_DF11-4DP-2DSA_2x02_P2.00mm_Vertical, symbol Connector_Generic:Conn_02x02_Counter_Clockwise
- added R1210, R1212: 470R, Resistor_SMD:R_0402_1005Metric, symbol Device:R_Small_US
- added U1203: AOZ13984DI-02, sub:DFN-12-1EP_3x3mm_P0.5mm_EP1.5x2.5mm, symbol sub_board:AOZ13984DI-02
- added U1205: 74LVC2G17, Package_TO_SOT_SMD:SOT-363_SC-70-6, symbol 74xGxx:74LVC2G17
- C1202, C1203, C1204: renamed from C?; footprint (none) -> Capacitor_SMD:C_0402_1005Metric
- C1205: renamed from C?; value 22uF, 63V, X7R -> 10uF, 63V, X7R; footprint (none) -> Capacitor_SMD:C_1210_3225Metric
- C1206, C1208: renamed from C?; footprint (none) -> Capacitor_SMD:C_0603_1608Metric
- C1210: renamed from C?; value 0.1uF, 50V -> 0.1uF, 63V; footprint (none) -> Capacitor_SMD:C_1206_3216Metric
- C1211, C1214: renamed from C?; value C_Small -> SOT; footprint (none) -> Capacitor_SMD:C_0603_1608Metric
- C1212: renamed from C?; value CP1 -> 100uF, 63V; footprint (none) -> sub:CP_MS10
- C1215: renamed from C?; value C_Small -> 330pF, 100V; footprint (none) -> Resistor_SMD:R_0805_2012Metric
- C1216: renamed from C?; value C_Small -> NIP; footprint (none) -> Capacitor_SMD:C_0603_1608Metric
- D1201: renamed from D?; footprint (none) -> Diode_SMD:D_SMC
- D1202: renamed from D?; value D -> 1N4148; footprint (none) -> Diode_SMD:D_SOD-123
- J1201, J1202: renamed from J?; footprint (none) -> Connector_Hirose:Hirose_DF13C_CL535-0404-8-51_1x04-1MP_P1.25mm_Vertical
- L1201: renamed from L?; footprint (none) -> sub:L_7447706150
- R1201, R1202, R1203, R1204, R1205, R1213: renamed from R?; footprint (none) -> Resistor_SMD:R_0402_1005Metric
- R1206: renamed from R?; footprint (none) -> Resistor_SMD:R_0603_1608Metric
- R1207, R1208: renamed from R?; footprint (none) -> Resistor_SMD:R_1206_3216Metric
- R1209: renamed from R?; value 4.7K -> 3K, 1/4W; footprint (none) -> Resistor_SMD:R_1206_3216Metric
- R1211: renamed from R?; value 4.7K -> NIP; footprint (none) -> Resistor_SMD:R_0603_1608Metric
- RL1201: renamed from RL?; value G2RL-2-ASI-DC5 -> EA2-5NJ; footprint Relay_THT:Relay_DPDT_Omron_G2RL -> sub:EA2-5NJ; symbol Relay:G2RL-2-ASI-DC5 -> sub_board:G2RL-2-DC5
- T1201: renamed from T?; value Transformer_SP_1S -> B78416A2232A003; footprint (none) -> sub:XFRMR_B78416
- U1201: renamed from U?; footprint (none) -> Package_DFN_QFN:DFN-14-1EP_3x4mm_P0.5mm_EP1.7x3.3mm
- U1202: renamed from U?; footprint (none) -> Package_TO_SOT_SMD:SOT-23-5
- U1204: renamed from U?; footprint (none) -> sub:WQFN-20
- gave numbers to parts that had none: 1
Connections:
- net i2c_master_scl is gone; now on net GND: J1202.2 (Pin_2)
- net +3V3: now also F1202.2, U1205.5 (VCC), U1205.5 (VCC); no longer J1201.1 (Pin_1)
- net +5V: now also RL1201.1 (+); no longer RL1201.8
- net +BATT: now also C1201.1, C1207.1, C1218.1, U1203.10 (Vin), U1203.9 (Vin); no longer J1202.1 (Pin_1)
- net GND: now also C1201.2, C1207.2, C1209.2, C1213.2, C1217.2, C1218.2, C1219.2, U1203.6 (gnd), U1205.2 (GND), U1205.2 (GND); no longer J1202.4 (Pin_4)
- net at C1205.1, D1201.1 (K), R1204.2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: now also C1219.1
- net at C1216.1, R1207.1, R1211.1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: now also RL1201.8; no longer RL1201.6
- net at RL1201.7: now also J1203.1 (Pin_1); no longer R1209.1
- net at RL1201.2: now also J1203.3 (Pin_3)
- net at RL1201.4: now also J1203.4 (Pin_4)
- net at D1202.2 (A), Q1201.3 (D): now also RL1201.10 (-); no longer RL1201.1
- net at R1209.2: now also RL1201.9, J1203.2 (Pin_2); no longer C1215.1
- net i2c_master_sda: no longer names the net of J1202.3 (Pin_3)
- net i2c_master_sda: now also R1212.1
- new net: F1202.1, J1201.1 (Pin_1)
- new net: F1201.1, J1202.1 (Pin_1)
- new net: J1202.4 (Pin_4), R1210.1
- new net: C1215.1, R1209.1
- new net: F1201.2, U1203.1 (Vout), U1203.2 (Vout)
- new net: C1209.1, U1203.4 (cap)
- new net: C1213.1, U1203.7 (ss)
- new net: R1210.2, U1205.6
- new net: C1217.1, R1212.2, U1205.3
- new net lidar_pwr: U1203.5 (en)
- new net lidar_rx: U1205.4
- new net lidar_tx: U1205.1
Other:
- moved on the sheet: J1201, J1202, Q1201, R1209, R1213
